File: matrix_slim.kicad_sch (KiCad schematic)
At the start: 66 parts, among them J2 C168688, SW1 PG1316M, SW10 PG1316S, SW11 PG1316S, SW12 PG1316S, SW13 PG1316S, SW14 PG1316S, SW15 PG1316M, SW16 PG1316M, SW17 PG1316S, SW18 PG1316M, SW2 PG1316M, SW3 PG1316M, SW4 PG1316M, SW5 PG1316M, SW6 PG1316S, SW7 PG1316S, SW8 PG1316S, SW9 PG1316S, U1 nRF52840, U2 BQ24075RGT, U3 XC6220B331MR, Y1 FC-12M, Y2 23MHz XRCGB32M000F1H50R0

Commit message: Added base setup
Parts:
- removed C1, C17, C18, C19: 100nF, Capacitor_SMD:C_0201_0603Metric, symbol Device:C
- removed C10, C14, C15, C9: 12pF, Capacitor_SMD:C_0201_0603Metric, symbol Device:C
- removed C11, C12: 1pF, Capacitor_SMD:C_0201_0603Metric, symbol Device:C
- removed C13: 1.5pF, Capacitor_SMD:C_0201_0603Metric, symbol Device:C
- removed C16, C21, C6: 1uF, Capacitor_SMD:C_0201_0603Metric, symbol Device:C
- removed C2: 100pF, Capacitor_SMD:C_0201_0603Metric, symbol Device:C
- removed C20, C22, C23, C4, C7, C8: 4.7uF, Capacitor_SMD:C_0201_0603Metric, symbol Device:C
- removed C24: 10uF, Capacitor_SMD:C_0201_0603Metric, symbol Device:C
- removed C25: 4.7nF, Capacitor_SMD:C_0201_0603Metric, symbol Device:C
- removed C3: 820pF, Capacitor_SMD:C_0201_0603Metric, symbol Device:C
- removed C5: 47nF, Capacitor_SMD:C_0201_0603Metric, symbol Device:C
- removed D1: RED, LED_SMD:LED_0201_0603Metric, symbol Device:LED
- removed D2: BLUE, LED_SMD:LED_0201_0603Metric, symbol Device:LED
- removed J2: C168688, custom_footprints:C168688, symbol MyLib:C168688
- removed JP1: Charge Boost, Jumper:SolderJumper-2_P1.3mm_Bridged2Bar_Pad1.0x1.5mm, symbol Jumper:Jumper_2_Open
- removed L1, L3: 10uH, Inductor_SMD:L_0201_0603Metric, symbol Device:L
- removed L2: 15nH, Inductor_SMD:L_0201_0603Metric, symbol Device:L
- removed L4: 3.9nH, Inductor_SMD:L_0201_0603Metric, symbol Device:L
- removed R1: 0, Resistor_SMD:R_0201_0603Metric, symbol Device:R
- removed R10, R11: 5.1k, Resistor_SMD:R_0201_0603Metric, symbol Device:R
- removed R2, R4, R5: 10k, Resistor_SMD:R_0201_0603Metric, symbol Device:R
- removed R3: 2k, Resistor_SMD:R_0201_0603Metric, symbol Device:R
- removed R6: 10M, Resistor_SMD:R_0201_0603Metric, symbol Device:R
- removed R7: 1k, Resistor_SMD:R_0201_0603Metric, symbol Device:R
- removed S1: MSK12C02, custom_footprints:MSK12C02, symbol MyLib:MSK12C02
- removed SW1, SW15, SW16, SW18, SW2, SW3, SW4, SW5: PG1316M, custom_footprints:CPG1316M01D02, symbol MyLib:PG1316M
- removed SW10, SW11, SW12, SW13, SW14, SW17, SW6, SW7, SW8, SW9: PG1316S, custom_footprints:CPG1316S01D02, symbol MyLib:PG1316S
- removed U1: nRF52840, Package_DFN_QFN:Nordic_AQFN-73-1EP_7x7mm_P0.5mm, symbol MCU_Nordic:nRF52840
- removed U2: BQ24075RGT, Package_DFN_QFN:VQFN-16-1EP_3x3mm_P0.5mm_EP1.6x1.6mm, symbol Battery_Management:BQ24075RGT
- removed U3: XC6220B331MR, Package_TO_SOT_SMD:SOT-23-5, symbol Regulator_Linear:XC6220B331MR
- removed Y1: FC-12M, Crystal:Crystal_SMD_3215-2Pin_3.2x1.5mm, symbol Device:Crystal
- removed Y2: 23MHz XRCGB32M000F1H50R0, custom_footprints:XRCGB32M000F1H01R0, symbol Device:Crystal_GND2
- added SW1, SW15, SW16, SW18, SW3, SW4, SW5, SW6: PG1316M, PG1316M:PG1316M, symbol PG1316M:PG1316M
- added SW10, SW11, SW12, SW13, SW14, SW17, SW2, SW7, SW8, SW9: PG1316S, PG1316S:PG1316S, symbol PG1316S:PG1316S
- added U1: NRF52840-CKAA-R, NRF52840-CKAA-R:NRF52840-CKAA-R, symbol NRF52840-CKAA-R:NRF52840-CKAA-R
Connections:
- net GND: now also SW1.2, SW10.2, SW11.2, SW12.2, SW13.2, SW14.2, SW15.2, SW16.2, SW17.2, SW18.2, SW2.2, SW3.2, SW4.2, SW5.2, SW6.2, SW7.2, SW8.2, SW9.2
- new net SGND: SW1.3 (SGND), SW10.3 (SGND), SW11.3 (SGND), SW12.3 (SGND), SW13.3 (SGND), SW14.3 (SGND), SW15.3 (SGND), SW16.3 (SGND), SW17.3 (SGND), SW18.3 (SGND), SW2.3 (SGND), SW3.3 (SGND), SW4.3 (SGND), SW5.3 (SGND), SW6.3 (SGND), SW7.3 (SGND), SW8.3 (SGND), SW9.3 (SGND)
- no-connect marks 7 -> 0
Other:
- note removed: "matrix slim"
